File: GOMA_V2.kicad_pcb (KiCad board)
At the start: 2 copper layers, 80 x 104.1 mm, 95 parts, among them J1 ch1 in, J10 ch3 in, J11 ch3 out, J12 Conn_01x07_Pin, J13 Conn_01x07_Socket, J14 ch4 in, J15 ch4 out, J16 Conn_01x08_Pin, J17 Conn_01x08_Socket, J18 Conn_02x05_Odd_Even, J19 Daisy out, J2 ch1 out, J3 Daisy in, J4 ch2 in, J5 ch2 out, J6 Conn_01x07_Pin, J7 Conn_01x07_Socket, J8 Conn_01x07_Pin, J9 Conn_01x07_Socket, SW1 SW_SPST, SW2 SW_SPST, SW3 SW_SPST, SW4 SW_SPST, U1 LM324, U2 LM324, U3 LM324, U4 LM324, U6 LM78L05_TO92

Commit message: ibom and kicad files
Other:
- board text added: "github.com/gunida v3 2025-08"
